File: Controls/controls/controls.kicad_sch (KiCad schematic)
At the start: 0 parts

Commit message: updated controls kicad
Parts:
- added SW1: SW_SPST, symbol Switch:SW_SPST
- added U1: MPU-6050, Sensor_Motion:InvenSense_QFN-24_4x4mm_P0.5mm, symbol Sensor_Motion:MPU-6050
- added U2: L298N, Package_TO_SOT_THT:TO-220-15_P2.54x5.08mm_StaggerOdd_Lead4.58mm_Vertical, symbol Driver_Motor:L298N
Connections:
- new net GND: U1.18 (GND), U2.8 (GND)
