File: Controls/controls KiCad/controls.kicad_sch (KiCad schematic)
At the start: 5 parts, among them U2 L298N

Commit message: Added notes to schematics
Other:
- note added: "We need 3 more of this, and add motors and Nano to schematic to show where it is connected."
Changed lines of the file:
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@@
 	(generator_version "9.0")
 	(paper "A4")
+	(text "We need 3 more of this, and add motors and Nano to schematic to show where it is connected. "
+		(exclude_from_sim no)
+		(at 115.316 160.528 0)
+		(effects
+			(font
+				(size 1.27 1.27)
+			)
+		)
+	)
 	(junction
 		(at 123.19 147.32)
