File: Controls/sensor and switch KiCad/sensor and switch.kicad_sch (KiCad schematic)
At the start: 5 parts, among them SW1 SW_SPST, U1 MPU-6050

Commit message: Added notes to schematics
Other:
- note added: "Potentially (probably) need more movement limit switches. I''l lyk at the meeting"
Changed lines of the file:
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@@
 	(generator_version "9.0")
 	(paper "A4")
+	(text "Potentially (probably) need more movement limit switches. I''l lyk at the meeting"
+		(exclude_from_sim no)
+		(at 116.332 138.176 0)
+		(effects
+			(font
+				(size 1.27 1.27)
+			)
+		)
+	)
 	(junction
 		(at 125.73 82.55)

Commit message: Updated minor note
Other:
- note added: "Absolutely no movement limit switches. Do need encoders though"
- note removed: "Potentially (probably) need more movement limit switches. I''l lyk at the meeting"
Changed lines of the file:
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@@
 	(generator_version "9.0")
 	(paper "A4")
-	(text "Potentially (probably) need more movement limit switches. I''l lyk at the meeting"
+	(text "Absolutely no movement limit switches. Do need encoders though"
 		(exclude_from_sim no)
 		(at 116.332 138.176 0)

Commit message: just some updates
Parts:
- removed R1: 2.2ohm, symbol Device:R_Small_US
- removed SW1: SW_SPST, symbol Switch:SW_SPST
- added U10, U3, U8, U9: ~, symbol Lunabotics 2025-26:SRX_Mag_Encoder
- added U2: ~, symbol Lunabotics 2025-26:Jetson_Nano
- added U4, U5, U6, U7: ~, symbol Lunabotics 2025-26:Spark_MAX_Motor_Controller
Connections:
- net GND: now also U10.10 (GND), U3.10 (GND), U8.10 (GND), U9.10 (GND)
- net +3.3V renamed Nano 3.3V
Other:
- note removed: "Absolutely no movement limit switches. Do need encoders though"
- moved on the sheet: U1

Commit message: Updated Control Schematic
Wired Motor Controller + Both Breakout Boards + Mag Encoder
Parts:
- removed U10, U8, U9: ~, symbol Lunabotics 2025-26:SRX_Mag_Encoder
- removed U2: ~, symbol Lunabotics 2025-26:Jetson_Nano
- removed U4, U7: ~, symbol Lunabotics 2025-26:Spark_MAX_Motor_Controller
- added U10, U14, U18, U9: ~, symbol Lunabotics 2025-26:Breakout_Board_Mag-Board
- added U11, U15, U19, U4: ~, symbol Lunabotics 2025-26:SRX_Mag_Encoder
- added U12, U16, U2: ~, symbol Lunabotics 2025-26:Spark_MAX_Motor_Controller
- added U13, U17, U7, U8: ~, symbol Lunabotics 2025-26:Breakout_Board_Max-Board
Connections:
- new net: U11.1 (3.3V), U11.10 (GND), U11.2 (5V), U11.3 (NC), U11.4 (FLMT), U11.5 (B), U11.6 (NC), U11.7 (A), U11.8 (RLMT), U11.9 (PWM), U9.11 (Data_Port_(10Pin))
- new net: U5.10 (Data_Port_(10Pin)), U8.12 (Data_Port_(10Pin))
- new net: U14.11 (Data_Port_(10Pin)), U15.1 (3.3V), U15.10 (GND), U15.2 (5V), U15.3 (NC), U15.4 (FLMT), U15.5 (B), U15.6 (NC), U15.7 (A), U15.8 (RLMT), U15.9 (PWM)
- new net: U17.10 (5.0V), U18.9 (5.0V)
- new net: U16.10 (Data_Port_(10Pin)), U17.12 (Data_Port_(10Pin))
- new net: U17.3 (P6), U18.4 (P7)
- new net: U17.5 (R_(Limit)), U18.6 (P5)
- new net: U17.9 (GND), U18.1 (GND)
- new net: U12.10 (Data_Port_(10Pin)), U13.12 (Data_Port_(10Pin))
- new net: U10.9 (5.0V), U7.10 (5.0V)
- new net: U6.10 (Data_Port_(10Pin)), U7.12 (Data_Port_(10Pin))
- new net: U10.4 (P7), U7.3 (P6)
- new net: U10.6 (P5), U7.5 (R_(Limit))
- new net: U10.1 (GND), U7.9 (GND)
- new net: U13.9 (GND), U14.1 (GND)
- new net: U13.3 (P6), U14.4 (P7)
- new net: U13.5 (R_(Limit)), U14.6 (P5)
- new net: U13.10 (5.0V), U14.9 (5.0V)
- new net: U8.9 (GND), U9.1 (GND)
- new net: U8.3 (P6), U9.4 (P7)
- new net: U8.5 (R_(Limit)), U9.6 (P5)
- new net: U8.10 (5.0V), U9.9 (5.0V)
- new net: U10.11 (Data_Port_(10Pin)), U4.1 (3.3V), U4.10 (GND), U4.2 (5V), U4.3 (NC), U4.4 (FLMT), U4.5 (B), U4.6 (NC), U4.7 (A), U4.8 (RLMT), U4.9 (PWM)
- new net: U18.11 (Data_Port_(10Pin)), U19.1 (3.3V), U19.10 (GND), U19.2 (5V), U19.3 (NC), U19.4 (FLMT), U19.5 (B), U19.6 (NC), U19.7 (A), U19.8 (RLMT), U19.9 (PWM)
Other:
- moved on the sheet: U1, U3
